Commit message: Day 6: semantic_objects rebuilt, and two geometry defects the checklist never listed
The June modules become a working ROS 2 package: dotted params, intrinsics
read from my_bot's calibration file (no 554.0 defaults left), extrinsics from
TF at startup (camera_link for yaw and origin, laser_frame for the range
origin), TF at the detection stamp with a spinning listener, a fail-closed
rotation gate on /diff_cont/odom, min_returns and max_spread rejection,
track-id association with expiry and a jump guard, a clear_landmarks service,
DELETEALL markers, saves on the publish timer and no restore on start.

Two things the checklist did not know: the extractor searched the scan at
image azimuths (right-positive) while the lidar is left-positive, so a box on
the image's right took its range from the robot's left; and the projector put
the point at the lidar's range from the camera's origin, a 9 cm constant. The
window is now mirrored into lidar angles and the camera ray is intersected
with the lidar range circle. 28 new tests; 139 pass.

The camera is mounted on the robot's RIGHT (user, 14 Sep): camera_offset_y is
now -0.03 in camera.xacro.

Makefile gains semantic, test, bridge, bridge-venv, ui, ui-deps.
landmark_tape_measure.py scores /semantic_landmarks against a taped truth.

Co-Authored-By: Claude Fable 5.1 <noreply@anthropic.com>
Claude-Session: https://claude.ai/code/session_01QheeTrrzt7Bef8sUtP6D89

File: src/my_bot/description/camera.xacro (robot description, xacro)
@@ -5,9 +5,11 @@
          at 640x480, RELIABLE QoS.
          THIS FILE IS THE CAMERA EXTRINSICS. Decision D-10: the semantic node
-         looks up base_link -> camera_optical_link from TF rather than reading
-         camera.dx/dy/yaw out of a params file, so this joint origin is the
-         single source and there is no second copy to drift against. The old
-         board's robot_params.yaml did carry those numbers and it did not
-         survive; nothing here is recovered from it.
+         looks up base_link -> camera_link (the x-forward MOUNT frame, not the
+         optical one: its 2D projector wants the mount's yaw, and the optical
+         frame's yaw is -90 deg) from TF rather than reading camera.dx/dy/yaw
+         out of a params file, so this joint origin is the single source and
+         there is no second copy to drift against. The old board's
+         robot_params.yaml did carry those numbers and it did not survive;
+         nothing here is recovered from it.
          MEASURED 2026-09-09 by tape measure, and expressed in the terms that
          were actually measured (height above the FLOOR, distance from the
@@ -16,5 +18,5 @@
          parented to chassis, so both properties add the base_link -> chassis
          offset back in.
-         camera_link lands at (0.05, 0.03, 0.167) in base_link. -->
+         camera_link lands at (0.05, -0.03, 0.167) in base_link. -->
     <!-- Height of the lens centre above the floor. The lidar sits at 0.22, so
          the camera is 2 cm BELOW the scan plane: an object the camera sees
@@ -30,10 +32,11 @@
     <xacro:property name="camera_offset_from_axle" value="0.05"/>
     <!-- Lateral offset from the robot centreline, POSITIVE LEFT (REP-103).
-         MAGNITUDE MEASURED (3 cm), SIDE ASSUMED LEFT. If the camera is
-         actually right of centre this must become -0.03. The error is small
-         and constant, so it will not look like a bug: every landmark lands
-         6 cm to one side, which reads as calibration slop rather than a sign
-         error. Confirm by eye before Day 6 and correct here, not downstream. -->
-    <xacro:property name="camera_offset_y" value="0.03"/>
+         MAGNITUDE MEASURED 9 Sep (3 cm). SIDE CONFIRMED 14 Sep BY THE USER:
+         the camera is mounted on the robot's RIGHT, so this is NEGATIVE.
+         It was +0.03 (left, assumed) from 9 to 14 Sep. The semantic node
+         reads this from TF (D-10) and intersects the camera's ray with the
+         lidar's range circle, so a wrong sign here moves every landmark by
+         the full 6 cm and reads as calibration slop, not as a bug. -->
+    <xacro:property name="camera_offset_y" value="-0.03"/>
     <!-- Mount tilt, in radians, POSITIVE NOSE-DOWN. Measured ~3 degrees UP,
          hence negative: a rotation of +p about +y sends the x-axis toward -z.
