Commit message: Odom said 0.9 mm, the floor said 10.9 cm: a 0.60% wheel asymmetry
calibrate_straight.py, 3 m closed loop at 0.10 m/s, marks sighted down
through the lidar puck centre, distance read as 5 tiles at nominal 600 mm.

The closed loop steers on ODOM lateral offset and ODOM yaw, so it drives
odom's ESTIMATE of the path straight. Odom held lateral to 0.9 mm; the robot
finished 10.9 cm right of the line with its heading turned the same way. That
gap cannot be anything but odometry bias: 4.07 deg of uncorrected yaw over
3 m, k_r - k_l = -0.005964.

Applied as per-side radius multipliers, not as an enc_counts_per_rev split.
Counts per rev is a property of the encoder disc and the gearbox and both
sides are the same parts; only tyre diameter can differ between wheels. Same
reasoning that rejected the old l:2473 r:2556 figures. diff_drive_controller
applies multipliers to the wheel commands too, so the robot drives straighter
rather than merely reporting better.

wheel_radius deliberately NOT changed. The same run suggests 0.03264, but
that is 5.2 mm over 3 m and the distance was COUNTED as five 600 mm tiles,
not taped -- grout makes tile pitch vary by more than the correction. The
uncertainty exceeds the correction, so applying it would record noise as a
calibration.

Also carries the by-hand wheel_separation 0.25168 / wheel_offset_y 0.12584
from earlier today, committed because an uncommitted calibration constant is
exactly what this project exists to stop losing. ITS PROVENANCE IS STILL NOT
RECORDED, and both comments now say so -- the old ones asserted 0.25 and
0.125 beside the new values, which is the prose-disagrees-with-values trap
that the encoder-split story already cost this project once.

Verification owed: re-run the 3 m loop, floor lateral should drop under 1 cm.

Co-Authored-By: Claude Opus 5 <noreply@anthropic.com>
Claude-Session: https://claude.ai/code/session_01FgDUpDpDSasDKec6gpYK2b

File: src/my_bot/description/robot_core.xacro (robot description, xacro)
@@ -24,6 +24,9 @@
          0.21/2 + 0.02 = 0.125. This value is exactly half of diff_cont's
          wheel_separation in config/my_controllers.yaml. Change one and you must
-         change the other, or odometry yaw drifts. -->
-    <xacro:property name="wheel_offset_y" value="0.125"/>
+         change the other, or odometry yaw drifts.
+         Raised to 0.12584 on 9 Sep to match wheel_separation 0.25168. The
+         pairing is correct, but see my_controllers.yaml: that separation
+         figure's provenance is not recorded. -->
+    <xacro:property name="wheel_offset_y" value="0.12584"/>
     <xacro:property name="wheel_offset_z" value="0.01"/>
     <!-- MEASURED: 38 mm, which is LARGER than the 34 mm drive wheels. The

Commit message: wheel_radius 0.03203 (5 m taped run, -2.0 %); calibrate_straight hint no longer uses the free radius 0.034
Co-Authored-By: Claude Opus 5.5 <noreply@anthropic.com>

File: src/my_bot/description/robot_core.xacro (robot description, xacro)
@@ -13,5 +13,5 @@
          this URDF. Change one and you must change the other, or the URDF's
          ground plane and lidar height drift away from the real robot. -->
-    <xacro:property name="wheel_radius" value="0.0327"/>
+    <xacro:property name="wheel_radius" value="0.03203"/>
     <xacro:property name="wheel_thickness" value="0.028"/>
     <xacro:property name="wheel_mass" value="0.05"/>

Commit message: wheel_radius back to 0.0327: the 0.03203 correction had the wrong sign for the map error
Co-Authored-By: Claude Opus 5.5 <noreply@anthropic.com>

File: src/my_bot/description/robot_core.xacro (robot description, xacro)
@@ -13,5 +13,5 @@
          this URDF. Change one and you must change the other, or the URDF's
          ground plane and lidar height drift away from the real robot. -->
-    <xacro:property name="wheel_radius" value="0.03203"/>
+    <xacro:property name="wheel_radius" value="0.0327"/>
     <xacro:property name="wheel_thickness" value="0.028"/>
     <xacro:property name="wheel_mass" value="0.05"/>
